Commit message: minor changes

File: src/setup/models/p3at/defs/pioneer3at.xacro (robot description, xacro)
@@ -5,5 +5,5 @@
        xmlns:xacro="http://ros.org/wiki/xacro"
 name="pioneer3at">
-<include filename="$(find setup)/defs/pioneer3at_body.xacro"/>
+<include filename="$(find setup)/models/p3at/defs/pioneer3at_body.xacro"/>
      <xacro:hokuyo_ust20lx laser_prefix="$(optenv LASER1_PREFIX base)" parent="$(optenv VECTOR_PARENT_LINK top_plate)">
         <origin xyz="$(optenv LASER1_XYZ 0.2 -0.1 0.02)" rpy="$(optenv LASER1_RPY 3.14159 0 0)" />

File: src/setup/models/p3at/defs/pioneer3at_body.xacro (robot description, xacro)
@@ -17,5 +17,5 @@
 			<origin xyz="0 0 0.177" rpy="0 0 0"/>
 			<geometry name="pioneer_geom">
-				<mesh filename="package://setup/meshes/chassis.stl"/>
+				<mesh filename="package://setup/models/p3at/meshes/chassis.stl"/>
 			</geometry>
 			<material name="ChassisRed">
@@ -26,5 +26,5 @@
 			<origin xyz="0 0 0.177" rpy="0 0 0"/>
 				<geometry>
-					<mesh filename="package://setup/meshes/chassis.stl"/>
+					<mesh filename="package://setup/models/p3at/meshes/chassis.stl"/>
 				</geometry>
 		</collision>
@@ -45,5 +45,5 @@
 			<origin xyz="0 0 0" rpy="0 0 0"/>
 			<geometry name="pioneer_geom">
-				<mesh filename="package://setup/meshes/top.stl"/>
+				<mesh filename="package://setup/models/p3at/meshes/top.stl"/>
 			</geometry>
 			<material name="TopBlack">
@@ -77,5 +77,5 @@
 			<origin xyz="0 0 0" rpy="0 0 0"/>
 			<geometry name="pioneer_geom">
-				<mesh filename="package://setup/meshes/front_sonar.stl"/>
+				<mesh filename="package://setup/models/p3at/meshes/front_sonar.stl"/>
 			</geometry>
 			<material name="SonarYellow">
@@ -108,5 +108,5 @@
 			<origin xyz="0 0 0" rpy="0 0 0"/>
 			<geometry name="pioneer_geom">
-				<mesh filename="package://setup/meshes/back_sonar.stl"/>
+				<mesh filename="package://setup/models/p3at/meshes/back_sonar.stl"/>
 			</geometry>
 			<material name="SonarYellow">
@@ -141,5 +141,5 @@
 		<origin xyz="0 0 0" rpy="0 0 0"/>
 		<geometry name="pioneer_geom">
-			<mesh filename="package://setup/meshes/axle.stl"/>
+			<mesh filename="package://setup/models/p3at/meshes/axle.stl"/>
 		</geometry>
 		<material name="AxleGrey">
@@ -172,5 +172,5 @@
 		<origin xyz="0 0 0" rpy="0 0 0"/>
 		<geometry name="pioneer_geom">
-			<mesh filename="package://setup/meshes/${suffix}_hubcap.stl"/>
+			<mesh filename="package://setup/models/p3at/meshes/${suffix}_hubcap.stl"/>
 		</geometry>
 		<material name="HubcapYellow">
@@ -203,5 +203,5 @@
 		<origin xyz="0 0 0" rpy="0 0 0"/>
 		<geometry name="pioneer_geom">
-			<mesh filename="package://setup/meshes/wheel.stl"/>
+			<mesh filename="package://setup/models/p3at/meshes/wheel.stl"/>
 		</geometry>
 		<material name="WheelBlack">
@@ -242,5 +242,5 @@
 		<origin xyz="0 0 0" rpy="0 0 0"/>
 		<geometry name="pioneer_geom">
-			<mesh filename="package://setup/meshes/axle.stl"/>
+			<mesh filename="package://setup/models/p3at/meshes/axle.stl"/>
 		</geometry>
 		<material name="AxleGrey">
@@ -251,5 +251,5 @@
 		<origin xyz="0 0 0" rpy="0 0 0"/>
 		<geometry>
-			<mesh filename="package://setup/meshes/axle.stl"/>
+			<mesh filename="package://setup/models/p3at/meshes/axle.stl"/>
 		</geometry>
 	</collision>
@@ -273,5 +273,5 @@
 		<origin xyz="0 0 0" rpy="0 0 0"/>
 		<geometry name="pioneer_geom">
-			<mesh filename="package://setup/meshes/${suffix}_hubcap.stl"/>
+			<mesh filename="package://setup/models/p3at/meshes/${suffix}_hubcap.stl"/>
 		</geometry>
 		<material name="HubcapYellow"/>
@@ -280,5 +280,5 @@
 		<origin xyz="0 0 0" rpy="0 0 0"/>
 		<geometry>
-			<mesh filename="package://setup/meshes/${suffix}_hubcap.stl"/>
+			<mesh filename="package://setup/models/p3at/meshes/${suffix}_hubcap.stl"/>
 		</geometry>
 	</collision>
@@ -302,5 +302,5 @@
 		<origin xyz="0 0 0" rpy="0 0 0"/>
 		<geometry name="pioneer_geom">
-			<mesh filename="package://setup/meshes/wheel.stl"/>
+			<mesh filename="package://setup/models/p3at/meshes/wheel.stl"/>
 		</geometry>
 		<material name="WheelBlack"/>
