Commit message: minor change

File: src/husky/husky_description/urdf/husky.urdf.xacro (robot description, xacro)
@@ -111,5 +111,5 @@
     </xacro:hokuyo_ust20lx>
     <xacro:pgr_flea3 camera_prefix="$(optenv LASER1_PREFIX base)" parent="$(optenv VECTOR_PARENT_LINK base)">
-       <origin xyz="$(optenv LASER1_XYZ 0 0 -0.05)" rpy="$(optenv LASER1_RPY 0 0 0)" />
+       <origin xyz="$(optenv LASER1_XYZ 0 0 -0.05)" rpy="$(optenv LASER1_RPY 3.14159 0 0)" />
    </xacro:pgr_flea3>
     </xacro:macro>
@@ -117,5 +117,4 @@
  <plugin name="skid_steer_drive_controller" filename="libgazebo_ros_skid_steer_drive.so">
     <updateRate>100.0</updateRate>
-    <robotNamespace></robotNamespace>
     <leftFrontJoint>front_left_wheel</leftFrontJoint>
     <rightFrontJoint>front_right_wheel</rightFrontJoint>
