Commit message: optimization work for move base

File: src/p3at_description/urdf/pioneer3at_body.xacro (robot description, xacro)
@@ -9,5 +9,5 @@
     <inertial>
       <mass value="14.0"/>
-      <origin xyz="0 0 0.177"/>
+      <origin xyz="0 0 0.085"/>
       <inertia ixx="0.14711667" ixy="0.0" ixz="0.0"
         iyy="0.334951167" iyz="0.0"

Commit message: updated center of mass

File: src/p3at_description/urdf/pioneer3at_body.xacro (robot description, xacro)
@@ -9,5 +9,5 @@
     <inertial>
       <mass value="14.0"/>
-      <origin xyz="0 0 0.085"/>
+      <origin xyz="0 0 0.04"/>
       <inertia ixx="0.14711667" ixy="0.0" ixz="0.0"
         iyy="0.334951167" iyz="0.0"
