Commit message: goto may 7th 2017 2300

File: src/p3at_description/urdf/pioneer3at.urdf.xacro (robot description, xacro)
@@ -9,7 +9,11 @@
   <xacro:include filename="$(find p3at_description)/urdf/hokuyo_utm30lx.urdf.xacro"/>
   <xacro:include filename="$(find p3at_description)/urdf/asus_camera.urdf.xacro" />
-  <xacro:hokuyo_utm30lx name="hokuyo" parent="base_link" ros_topic="hokuyo" update_rate="25" ray_count="720" min_angle="130" max_angle="-130" >   <!--raycount=1040  updaterate=30-->
+  <xacro:include filename="$(find p3at_description)/urdf/velodyne.urdf.xacro"/>
+ <!--xacro:hokuyo_utm30lx name="hokuyo" parent="base_link" ros_topic="hokuyo" update_rate="25" ray_count="720" min_angle="130" max_angle="-130" >   <comment raycount=1040  updaterate=30 comment>
     <origin xyz="0.13 0 0.32" rpy="0 0 0"/>
-  </xacro:hokuyo_utm30lx>
+  </xacro:hokuyo_utm30lx-->
+  <xacro:rotating_velodyne name="hokuyo" parent="base_link" ros_topic="hokuyo" update_rate="25" ray_count="360" min_angle="160" max_angle="-160" >
+    <origin xyz="0.13 0 0.32" rpy="0 0 0"/>
+  </xacro:rotating_velodyne>
   <xacro:asus_camera name="camera" parent="base_link">
 	                <origin xyz="0.065 0.0 0.43" rpy="0 0 0"/>

Commit message: theraml camera added.

File: src/p3at_description/urdf/pioneer3at.urdf.xacro (robot description, xacro)
@@ -9,4 +9,5 @@
   <xacro:include filename="$(find p3at_description)/urdf/hokuyo_utm30lx.urdf.xacro"/>
   <xacro:include filename="$(find p3at_description)/urdf/asus_camera.urdf.xacro" />
+  <xacro:include filename="$(find p3at_description)/urdf/thermal_camera.urdf.xacro" />
   <!--xacro:include filename="$(find p3at_description)/urdf/velodyne.urdf.xacro"/>
 <xacro:rotating_velodyne name="hokuyo" parent="base_link" ros_topic="hokuyo" update_rate="25" ray_count="360" min_angle="160" max_angle="-160" >
@@ -17,5 +18,8 @@
   </xacro:hokuyo_utm30lx>
   <xacro:asus_camera name="camera" parent="base_link">
-	                <origin xyz="0.065 0.0 0.43" rpy="0 0 0"/>
+	                <origin xyz="0.065 0.0 0.45" rpy="0 0 0"/>
   </xacro:asus_camera>
+  <xacro:flir_a35_camera name="thermal" parent="base_link">
+                  <origin xyz="0.105 0.0 0.40" rpy="0 0 0"/>
+  </xacro:flir_a35_camera>
 </robot>

Commit message: simple codes before iranopen2018

File: src/p3at_description/urdf/pioneer3at.urdf.xacro (robot description, xacro)
@@ -9,5 +9,4 @@
   <xacro:include filename="$(find p3at_description)/urdf/hokuyo_utm30lx.urdf.xacro"/>
   <xacro:include filename="$(find p3at_description)/urdf/asus_camera.urdf.xacro" />
-  <xacro:include filename="$(find p3at_description)/urdf/thermal_camera.urdf.xacro" />
   <!--xacro:include filename="$(find p3at_description)/urdf/velodyne.urdf.xacro"/>
 <xacro:rotating_velodyne name="hokuyo" parent="base_link" ros_topic="hokuyo" update_rate="25" ray_count="360" min_angle="160" max_angle="-160" >
@@ -18,8 +17,5 @@
   </xacro:hokuyo_utm30lx>
   <xacro:asus_camera name="camera" parent="base_link">
-	                <origin xyz="0.065 0.0 0.45" rpy="0 0 0"/>
+	                <origin xyz="0.095 0.0 0.38" rpy="0 0 0"/>
   </xacro:asus_camera>
-  <xacro:flir_a35_camera name="thermal" parent="base_link">
-                  <origin xyz="0.105 0.0 0.40" rpy="0 0 0"/>
-  </xacro:flir_a35_camera>
 </robot>

File: src/p3at_description/urdf/pioneer3at_body.xacro (robot description, xacro)
@@ -141,5 +141,5 @@
   <gazebo>
     <plugin name="skid_steer_drive_controller" filename="libgazebo_ros_skid_steer_drive.so">
-      <updateRate>100.0</updateRate>
+      <updateRate>5.0</updateRate>
       <!--robotNamespace>$(arg robot_name)</robotNamespace-->
       <leftFrontJoint>p3at_front_left_wheel_joint</leftFrontJoint>

File: src/p3at_description/urdf/thermal_camera.urdf.xacro (robot description, xacro)
@@ -61,5 +61,5 @@
           </clip>
         </camera>
-        <plugin name="thermal_camera_controller" filename="libgazebo_ros_thermal_camera.so">
+        <plugin name="thermal_camera_controller" filename="package://hector_gazebo_thermal_camera/libgazebo_ros_thermal_camera_pink.so">
           <alwaysOn>true</alwaysOn>
           <updateRate>10</updateRate>

Commit message: thermal camera removed

File: src/p3at_description/urdf/pioneer3at.urdf.xacro (robot description, xacro)
@@ -9,5 +9,4 @@
   <xacro:include filename="$(find p3at_description)/urdf/hokuyo_utm30lx.urdf.xacro"/>
   <xacro:include filename="$(find p3at_description)/urdf/asus_camera.urdf.xacro" />
-  <xacro:include filename="$(find p3at_description)/urdf/thermal_camera.urdf.xacro" />
   <!--xacro:include filename="$(find p3at_description)/urdf/velodyne.urdf.xacro"/>
 <xacro:rotating_velodyne name="hokuyo" parent="base_link" ros_topic="hokuyo" update_rate="25" ray_count="360" min_angle="160" max_angle="-160" >
@@ -20,6 +19,3 @@
 	                <origin xyz="0.065 0.0 0.45" rpy="0 0 0"/>
   </xacro:asus_camera>
-  <xacro:flir_a35_camera name="thermal" parent="base_link">
-                  <origin xyz="0.105 0.0 0.40" rpy="0 0 0"/>
-  </xacro:flir_a35_camera>
 </robot>
